Commit message: add imu offsets for oak-d-lr

File: depthai_descriptions/urdf/include/base_macro.urdf.xacro (robot description, xacro)
@@ -56,12 +56,31 @@
             <xacro:property name="imu_y" value="0.0" />
         </xacro:if>
-        <xacro:if value="${has_imu}">
-            <link name="${camera_name}_imu_frame" />
-            <joint name="${camera_name}_imu_joint" type="fixed">
-                <parent link="${base_frame}"/>
-                <child link="${camera_name}_imu_frame"/>
-                <origin xyz="${imu_offset_x} ${imu_offset_y} ${imu_offset_z}" rpy="${imu_r} ${imu_p} ${imu_y}" />
-            </joint>
+        <!-- offsets are relative to left camera frame https://github.com/luxonis/depthai-boards/blob/adding_IMU_tmp/boards/OAK-D-LR.json -->
+        <xacro:if value="${model == 'OAK-D-LR'}">
+            <xacro:property name="imu_offset_x" value="12.1465" />
+            <xacro:property name="imu_offset_y" value="0.0" />
+            <xacro:property name="imu_offset_z" value="-1.2616" />
+            <xacro:property name="imu_r" value="0.0" />
+            <xacro:property name="imu_p" value="0.0" />
+            <xacro:property name="imu_y" value="0.0" />
+            <xacro:if value="${has_imu}">
+              <link name="${camera_name}_imu_frame" />
+              <joint name="${camera_name}_imu_joint" type="fixed">
+                  <parent link="${camera_name}_left_camera_frame"/>
+                  <child link="${camera_name}_imu_frame"/>
+                  <origin xyz="${imu_offset_x} ${imu_offset_y} ${imu_offset_z}" rpy="${imu_r} ${imu_p} ${imu_y}" />
+              </joint>
+            </xacro:if>
         </xacro:if>
+        <xacro:unless value="${model == 'OAK-D-LR'}">
+          <xacro:if value="${has_imu}">
+              <link name="${camera_name}_imu_frame" />
+              <joint name="${camera_name}_imu_joint" type="fixed">
+                  <parent link="${base_frame}"/>
+                  <child link="${camera_name}_imu_frame"/>
+                  <origin xyz="${imu_offset_x} ${imu_offset_y} ${imu_offset_z}" rpy="${imu_r} ${imu_p} ${imu_y}" />
+              </joint>
+          </xacro:if>
+        </xacro:unless>
     </xacro:macro>
 </robot>

Commit message: depthai_descriptions: change mm to meters for imu link

File: depthai_descriptions/urdf/include/base_macro.urdf.xacro (robot description, xacro)
@@ -58,7 +58,7 @@
         <!-- offsets are relative to left camera frame https://github.com/luxonis/depthai-boards/blob/adding_IMU_tmp/boards/OAK-D-LR.json -->
         <xacro:if value="${model == 'OAK-D-LR'}">
-            <xacro:property name="imu_offset_x" value="12.1465" />
+            <xacro:property name="imu_offset_x" value="0.0121465" />
             <xacro:property name="imu_offset_y" value="0.0" />
-            <xacro:property name="imu_offset_z" value="-1.2616" />
+            <xacro:property name="imu_offset_z" value="-0.0012616" />
             <xacro:property name="imu_r" value="0.0" />
             <xacro:property name="imu_p" value="0.0" />

Commit message: depthai_descriptions: adjustOAK-D-LR IMU translation and rotation

File: depthai_descriptions/urdf/include/base_macro.urdf.xacro (robot description, xacro)
@@ -58,9 +58,9 @@
         <!-- offsets are relative to left camera frame https://github.com/luxonis/depthai-boards/blob/adding_IMU_tmp/boards/OAK-D-LR.json -->
         <xacro:if value="${model == 'OAK-D-LR'}">
-            <xacro:property name="imu_offset_x" value="0.0121465" />
+            <xacro:property name="imu_offset_x" value="-0.0121465" />
             <xacro:property name="imu_offset_y" value="0.0" />
             <xacro:property name="imu_offset_z" value="-0.0012616" />
-            <xacro:property name="imu_r" value="0.0" />
-            <xacro:property name="imu_p" value="0.0" />
+            <xacro:property name="imu_r" value="${M_PI}" />
+            <xacro:property name="imu_p" value="${M_PI/2.0}" />
             <xacro:property name="imu_y" value="0.0" />
             <xacro:if value="${has_imu}">

Commit message: depthai_descriptions: fix imu rpy

File: depthai_descriptions/urdf/include/base_macro.urdf.xacro (robot description, xacro)
@@ -61,7 +61,7 @@
             <xacro:property name="imu_offset_y" value="0.0" />
             <xacro:property name="imu_offset_z" value="-0.0012616" />
-            <xacro:property name="imu_r" value="${M_PI}" />
-            <xacro:property name="imu_p" value="${M_PI/2.0}" />
-            <xacro:property name="imu_y" value="0.0" />
+            <xacro:property name="imu_r" value="${-M_PI/2.0}" />
+            <xacro:property name="imu_p" value="0.0" />
+            <xacro:property name="imu_y" value="${-M_PI/2.0}" />
             <xacro:if value="${has_imu}">
               <link name="${camera_name}_imu_frame" />
